File: espDash.sch (EAGLE design)
At the start: 13 parts

Commit message: 5 button
Added a button
Parts:
- added LED5: (no value), led:LED5MM
- added R5: (no value), rcl:R-EU_0207/10
- added S1: (no value), switch-omron:40-XX
- added S2: (no value), switch:M251
- added SL1, SL2: (no value), con-amp-quick:M15
Connections:
- new net N$14: LED5.A, R5.1
- net +3V3: now also SL2.11; no longer U$1.3V3@0
- net GND: now also LED5.C, S1.S, S1.S1, SL1.2; no longer U$1.GND@3
- net N$1: now also SL1.14; no longer U$1.D1
- net N$2: now also SL1.13; no longer U$1.D2
- net N$3: now also SL1.12; no longer U$1.D3
- net N$4: now also SL1.11; no longer U$1.D4
- net N$5: now also SL1.8; no longer U$1.D5
- net N$6: now also SL1.7; no longer U$1.D6
- net N$7: now also SL1.6; no longer U$1.D7
- net N$8: now also SL1.5; no longer U$1.D8
Other:
- moved on the sheet: U$1
Changed lines of the file:
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@@
 <layers>
 <layer number="1" name="Top" color="4" fill="1" visible="no" active="no"/>
+<layer number="2" name="Route2" color="1" fill="3" visible="no" active="no"/>
+<layer number="3" name="Route3" color="4" fill="3" visible="no" active="no"/>
+<layer number="4" name="Route4" color="1" fill="4" visible="no" active="no"/>
+<layer number="5" name="Route5" color="4" fill="4" visible="no" active="no"/>
+<layer number="6" name="Route6" color="1" fill="8" visible="no" active="no"/>
+<layer number="7" name="Route7" color="4" fill="8" visible="no" active="no"/>
+<layer number="8" name="Route8" color="1" fill="2" visible="no" active="no"/>
+<layer number="9" name="Route9" color="4" fill="2" visible="no" active="no"/>
+<layer number="10" name="Route10" color="1" fill="7" visible="no" active="no"/>
+<layer number="11" name="Route11" color="4" fill="7" visible="no" active="no"/>
+<layer number="12" name="Route12" color="1" fill="5" visible="no" active="no"/>
+<layer number="13" name="Route13" color="4" fill="5" visible="no" active="no"/>
+<layer number="14" name="Route14" color="1" fill="6" visible="no" active="no"/>
+<layer number="15" name="Route15" color="4" fill="6" visible="no" active="no"/>
 <layer number="16" name="Bottom" color="1" fill="1" visible="no" active="no"/>
 <layer number="17" name="Pads" color="2" fill="1" visible="no" active="no"/>
@@
 <part name="LED3" library="led" deviceset="LED" device="5MM"/>
 <part name="LED4" library="led" deviceset="LED" device="5MM"/>
-<part name="+3V1" library="supply1" deviceset="+3V3" device=""/>
 <part name="S5" library="switch-omron" deviceset="40-XX" device=""/>
 <part name="S6" library="switch-omron" deviceset="40-XX" device=""/>
@@
 <part name="GND9" library="supply1" deviceset="GND" device=""/>
 <part name="GND10" library="supply1" deviceset="GND" device=""/>
+<part name="SL1" library="con-amp-quick" deviceset="M15" device=""/>
+<part name="R5" library="rcl" deviceset="R-EU_" device="0207/10"/>
+<part name="LED5" library="led" deviceset="LED" device="5MM"/>
+<part name="GND1" library="supply1" deviceset="GND" device=""/>
+<part name="S1" library="switch-omron" deviceset="40-XX" device=""/>
+<part name="GND11" library="supply1" deviceset="GND" device=""/>
+<part name="SL2" library="con-amp-quick" deviceset="M15" device=""/>
+<part name="+3V2" library="supply1" deviceset="+3V3" device=""/>
+<part name="S2" library="switch" deviceset="M251" device=""/>
 </parts>
 <sheets>
@@
 </plain>
 <instances>
-<instance part="U$1" gate="G$1" x="5.08" y="58.42"/>
+<instance part="U$1" gate="G$1" x="-10.16" y="58.42"/>
 <instance part="R1" gate="G$1" x="38.1" y="40.64" rot="R90"/>
 <instance part="R2" gate="G$1" x="50.8" y="40.64" rot="R90"/>
@@
 <instance part="LED3" gate="G$1" x="63.5" y="25.4"/>
 <instance part="LED4" gate="G$1" x="76.2" y="25.4"/>
-<instance part="+3V1" gate="G$1" x="-30.48" y="50.8" rot="R90"/>
 <instance part="S5" gate="1" x="35.56" y="88.9"/>
 <instance part="S6" gate="1" x="48.26" y="88.9"/>
@@
 <instance part="GND9" gate="1" x="76.2" y="12.7"/>
 <instance part="GND10" gate="1" x="30.48" y="43.18" rot="R90"/>
+<instance part="SL1" gate="G$1" x="15.24" y="58.42"/>
+<instance part="R5" gate="G$1" x="88.9" y="40.64" rot="R90"/>
+<instance part="LED5" gate="G$1" x="88.9" y="25.4"/>
+<instance part="GND1" gate="1" x="88.9" y="12.7"/>
+<instance part="S1" gate="1" x="86.36" y="88.9"/>
+<instance part="GND11" gate="1" x="88.9" y="106.68" rot="R180"/>
+<instance part="SL2" gate="G$1" x="-35.56" y="58.42" rot="R180"/>
+<instance part="+3V2" gate="G$1" x="-48.26" y="50.8" rot="R90"/>
+<instance part="S2" gate="1" x="12.7" y="93.98"/>
 </instances>
 <busses>
@@
 <net name="N$1" class="0">
 <segment>
-<pinref part="U$1" gate="G$1" pin="D1"/>
 <pinref part="S5" gate="1" pin="P"/>
-<wire x1="22.86" y1="73.66" x2="35.56" y2="73.66" width="0.1524" layer="91"/>
+<wire x1="20.32" y1="73.66" x2="35.56" y2="73.66" width="0.1524" layer="91"/>
 <wire x1="35.56" y1="73.66" x2="35.56" y2="83.82" width="0.1524" layer="91"/>
+<pinref part="SL1" gate="G$1" pin="14"/>
 </segment>
 </net>
 <net name="N$2" class="0">
 <segment>
-<pinref part="U$1" gate="G$1" pin="D2"/>
 <pinref part="S6" gate="1" pin="P"/>
-<wire x1="22.86" y1="71.12" x2="48.26" y2="71.12" width="0.1524" layer="91"/>
+<wire x1="20.32" y1="71.12" x2="48.26" y2="71.12" width="0.1524" layer="91"/>
 <wire x1="48.26" y1="71.12" x2="48.26" y2="83.82" width="0.1524" layer="91"/>
+<pinref part="SL1" gate="G$1" pin="13"/>
 </segment>
 </net>
 <net name="N$3" class="0">
 <segment>
-<pinref part="U$1" gate="G$1" pin="D3"/>
 <pinref part="S7" gate="1" pin="P"/>
-<wire x1="22.86" y1="68.58" x2="60.96" y2="68.58" width="0.1524" layer="91"/>
+<wire x1="20.32" y1="68.58" x2="60.96" y2="68.58" width="0.1524" layer="91"/>
 <wire x1="60.96" y1="68.58" x2="60.96" y2="83.82" width="0.1524" layer="91"/>
+<pinref part="SL1" gate="G$1" pin="12"/>
 </segment>
 </net>
@@
 <pinref part="S8" gate="1" pin="P"/>
 <wire x1="73.66" y1="66.04" x2="73.66" y2="83.82" width="0.1524" layer="91"/>
-<pinref part="U$1" gate="G$1" pin="D4"/>
-<wire x1="22.86" y1="66.04" x2="73.66" y2="66.04" width="0.1524" layer="91"/>
+<pinref part="SL1" gate="G$1" pin="11"/>
+<wire x1="20.32" y1="66.04" x2="73.66" y2="66.04" width="0.1524" layer="91"/>
 </segment>
 </net>
 <net name="N$5" class="0">
 <segment>
-<pinref part="U$1" gate="G$1" pin="D5"/>
 <pinref part="R1" gate="G$1" pin="2"/>
-<wire x1="22.86" y1="58.42" x2="38.1" y2="58.42" width="0.1524" layer="91"/>
+<wire x1="20.32" y1="58.42" x2="38.1" y2="58.42" width="0.1524" layer="91"/>
 <wire x1="38.1" y1="58.42" x2="38.1" y2="45.72" width="0.1524" layer="91"/>
+<pinref part="SL1" gate="G$1" pin="8"/>
 </segment>
 </net>
 <net name="N$6" class="0">
 <segment>
-<pinref part="U$1" gate="G$1" pin="D6"/>
 <pinref part="R2" gate="G$1" pin="2"/>
-<wire x1="22.86" y1="55.88" x2="50.8" y2="55.88" width="0.1524" layer="91"/>
+<wire x1="20.32" y1="55.88" x2="50.8" y2="55.88" width="0.1524" layer="91"/>
 <wire x1="50.8" y1="55.88" x2="50.8" y2="45.72" width="0.1524" layer="91"/>
+<pinref part="SL1" gate="G$1" pin="7"/>
 </segment>
 </net>
 <net name="N$7" class="0">
 <segment>
-<pinref part="U$1" gate="G$1" pin="D7"/>
 <pinref part="R3" gate="G$1" pin="2"/>
-<wire x1="22.86" y1="53.34" x2="63.5" y2="53.34" width="0.1524" layer="91"/>
+<wire x1="20.32" y1="53.34" x2="63.5" y2="53.34" width="0.1524" layer="91"/>
 <wire x1="63.5" y1="53.34" x2="63.5" y2="45.72" width="0.1524" layer="91"/>
+<pinref part="SL1" gate="G$1" pin="6"/>
 </segment>
 </net>
 <net name="N$8" class="0">
 <segment>
-<pinref part="U$1" gate="G$1" pin="D8"/>
 <pinref part="R4" gate="G$1" pin="2"/>
-<wire x1="22.86" y1="50.8" x2="76.2" y2="50.8" width="0.1524" layer="91"/>
+<wire x1="20.32" y1="50.8" x2="76.2" y2="50.8" width="0.1524" layer="91"/>
 <wire x1="76.2" y1="50.8" x2="76.2" y2="45.72" width="0.1524" layer="91"/>
+<pinref part="SL1" gate="G$1" pin="5"/>
 </segment>
 </net>
@@
 </segment>
 <segment>
-<pinref part="U$1" gate="G$1" pin="GND@3"/>
 <pinref part="GND10" gate="1" pin="GND"/>
-<wire x1="22.86" y1="43.18" x2="27.94" y2="43.18" width="0.1524" layer="91"/>
+<pinref part="SL1" gate="G$1" pin="2"/>
+<wire x1="20.32" y1="43.18" x2="27.94" y2="43.18" width="0.1524" layer="91"/>
+</segment>
+<segment>
+<pinref part="LED5" gate="G$1" pin="C"/>
+<pinref part="GND1" gate="1" pin="GND"/>
+<wire x1="88.9" y1="20.32" x2="88.9" y2="15.24" width="0.1524" layer="91"/>
+</segment>
+<segment>
+<pinref part="S1" gate="1" pin="S1"/>
+<pinref part="GND11" gate="1" pin="GND"/>
+<wire x1="88.9" y1="93.98" x2="88.9" y2="96.52" width="0.1524" layer="91"/>
+<pinref part="S1" gate="1" pin="S"/>
+<wire x1="88.9" y1="96.52" x2="88.9" y2="104.14" width="0.1524" layer="91"/>
+<wire x1="86.36" y1="93.98" x2="86.36" y2="96.52" width="0.1524" layer="91"/>
+<wire x1="86.36" y1="96.52" x2="88.9" y2="96.52" width="0.1524" layer="91"/>
+<junction x="88.9" y="96.52"/>
 </segment>
 </net>
@@
 </segment>
 </net>
-<net name="+3V3" class="0">
-<segment>
-<pinref part="U$1" gate="G$1" pin="3V3@0"/>
-<pinref part="+3V1" gate="G$1" pin="+3V3"/>
-<wire x1="-12.7" y1="50.8" x2="-27.94" y2="50.8" width="0.1524" layer="91"/>
-</segment>
-</net>
 <net name="N$10" class="0">
 <segment>
@@
 </segment>
 </net>
+<net name="N$14" class="0">
+<segment>
+<pinref part="R5" gate="G$1" pin="1"/>
+<pinref part="LED5" gate="G$1" pin="A"/>
+<wire x1="88.9" y1="35.56" x2="88.9" y2="27.94" width="0.1524" layer="91"/>
+</segment>
+</net>
+<net name="+3V3" class="0">
+<segment>
+<pinref part="+3V2" gate="G$1" pin="+3V3"/>
+<pinref part="SL2" gate="G$1" pin="11"/>
+<wire x1="-45.72" y1="50.8" x2="-40.64" y2="50.8" width="0.1524" layer="91"/>
+</segment>
+</net>
